File: pcb/plate/krunchboard-plate.kicad_pcb (KiCad board)
At the start: 2 copper layers, 377.7 x 126.1 mm, 0 parts

Commit message: updated plate files
Changed lines of the file:
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@@
 			(layer "F.SilkS"
 				(type "Top Silk Screen")
+				(color "Black")
 			)
 			(layer "F.Paste"
@@
 			(layer "F.Mask"
 				(type "Top Solder Mask")
+				(color "White")
 				(thickness 0.01)
 			)
@@
 			(layer "dielectric 1"
 				(type "core")
+				(color "FR4 natural")
 				(thickness 1.51)
 				(material "FR4")
@@
 			(layer "B.Mask"
 				(type "Bottom Solder Mask")
+				(color "White")
 				(thickness 0.01)
 			)
@@
 			(layer "B.SilkS"
 				(type "Bottom Silk Screen")
+				(color "Black")
 			)
 			(copper_finish "None")
@@
 		(net 0)
 		(net_name "")
-		(layers "*.SilkS")
+		(layers "*.Mask")
 		(hatch edge 0.5)
 		(connect_pads
