File: kicad-pcb/plate/krunchboard-plate.kicad_pcb (KiCad board)
At the start: 2 copper layers, 448.2 x 159.3 mm, 12 parts

Commit message: final v1 pcb revision, plate update
Parts:
- moved REF** 12.5 mm to (22.4, 9.94)
- moved REF** 12.4 mm to (22.3, 159.2)
- moved REF** 12.1 mm to (436.0, 9.94)
- moved REF** 12.1 mm to (436.0, 159.2)
- moved REF** 0.11 mm to (229.1, 10.0)
- moved REF** 0.08 mm to (229.1, 159.1)
Other:
- board size 448.2 x 159.3 mm -> 434.2 x 159.3 mm
Changed lines of the file:
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@@
 	(footprint "MountingHole:MountingHole_3.2mm_M3"
 		(layer "F.Cu")
-		(at 228.988848 10)
+		(at 229.1 10)
 		(descr "Mounting Hole 3.2mm, no annular, M3")
 		(tags "mounting hole 3.2mm no annular m3")
@@
 	(footprint "MountingHole:MountingHole_3.2mm_M3"
 		(layer "F.Cu")
-		(at 448.0677 159.141)
+		(at 436 159.2)
 		(descr "Mounting Hole 3.2mm, no annular, M3")
 		(tags "mounting hole 3.2mm no annular m3")
@@
 	(footprint "MountingHole:MountingHole_3.2mm_M3"
 		(layer "F.Cu")
-		(at 229.18 159.13)
+		(at 229.1 159.13)
 		(descr "Mounting Hole 3.2mm, no annular, M3")
 		(tags "mounting hole 3.2mm no annular m3")
@@
 	(footprint "MountingHole:MountingHole_3.2mm_M3"
 		(layer "F.Cu")
-		(at 9.91 159.140984)
+		(at 22.3 159.2)
 		(descr "Mounting Hole 3.2mm, no annular, M3")
 		(tags "mounting hole 3.2mm no annular m3")
@@
 	(footprint "MountingHole:MountingHole_3.2mm_M3"
 		(layer "F.Cu")
-		(at 9.91 9.88)
+		(at 22.4 9.939016)
 		(descr "Mounting Hole 3.2mm, no annular, M3")
 		(tags "mounting hole 3.2mm no annular m3")
@@
 	(footprint "MountingHole:MountingHole_3.2mm_M3"
 		(layer "F.Cu")
-		(at 448.0677 9.88)
+		(at 436 9.939)
 		(descr "Mounting Hole 3.2mm, no annular, M3")
 		(tags "mounting hole 3.2mm no annular m3")
@@
 		(embedded_fonts no)
 	)
+	(gr_rect
+		(start 411.4379 86.8929)
+		(end 425.1279 92.9771)
+		(stroke
+			(width 0.05)
+			(type solid)
+		)
+		(fill no)
+		(layer "Cmts.User")
+	)
 	(gr_line
 		(start 85.45 41.7125)
@@
 		(layer "Edge.Cuts")
 	)
+	(gr_arc
+		(start 16.9 164.140984)
+		(mid 13.364466 162.676518)
+		(end 11.9 159.140984)
+		(stroke
+			(width 0.05)
+			(type default)
+		)
+		(layer "Edge.Cuts")
+	)
 	(gr_line
 		(start 380.225 109.175)
@@
 		(layer "Edge.Cuts")
 	)
-	(gr_rect
-		(start 411.4379 86.8929)
-		(end 425.1279 92.9771)
-		(stroke
-			(width 0.05)
-			(type default)
-		)
-		(fill no)
-		(layer "Edge.Cuts")
-	)
 	(gr_arc
 		(start 44.18125 122.175)
@@
 	)
 	(gr_arc
-		(start 4.91 9.88)
-		(mid 6.374466 6.344466)
-		(end 9.91 4.88)
-		(stroke
-			(width 0.05)
-			(type default)
-		)
-		(layer "Edge.Cuts")
-	)
-	(gr_arc
 		(start 332.3125 84.075)
 		(mid 332.166053 84.428553)
@@
 	)
 	(gr_line
-		(start 9.91 4.88)
-		(end 448.067695 4.88)
-		(stroke
-			(width 0.05)
-			(type default)
-		)
-		(layer "Edge.Cuts")
-	)
-	(gr_line
 		(start 60.85 52.025)
 		(end 60.85 65.025)
@@
 	)
 	(gr_arc
+		(start 441.075 4.88)
+		(mid 444.610534 6.344466)
+		(end 446.075 9.88)
+		(stroke
+			(width 0.05)
+			(type default)
+		)
+		(layer "Edge.Cuts")
+	)
+	(gr_arc
 		(start 271.1875 103.625)
 		(mid 270.833947 103.478553)
@@
 	)
 	(gr_arc
+		(start 11.9 9.88)
+		(mid 13.364466 6.344466)
+		(end 16.9 4.88)
+		(stroke
+			(width 0.05)
+			(type default)
+		)
+		(layer "Edge.Cuts")
+	)
+	(gr_arc
 		(start 179.4125 108.675)
 		(mid 179.766053 108.821447)
@@
 		(layer "Edge.Cuts")
 	)
+	(gr_rect
+		(start 402.0058 40.64)
+		(end 443.3062 141.6822)
+		(stroke
+			(width 0.05)
+			(type default)
+		)
+		(fill no)
+		(layer "Edge.Cuts")
+	)
 	(gr_arc
 		(start 351.3625 65.025)
@@
 		(layer "Edge.Cuts")
 	)
-	(gr_arc
-		(start 9.91 164.140984)
-		(mid 6.374466 162.676518)
-		(end 4.91 159.140984)
-		(stroke
-			(width 0.05)
-			(type default)
-		)
-		(layer "Edge.Cuts")
-	)
 	(gr_rect
 		(start 378.8504 25.3029)
-		(end 395.5004 43.8529)
+		(end 394.9924 43.8529)
 		(stroke
 			(width 0.05)
@@
 		(layer "Edge.Cuts")
 	)
+	(gr_line
+		(start 16.9 4.88)
+		(end 441.075 4.88)
+		(stroke
+			(width 0.05)
+			(type default)
+		)
+		(layer "Edge.Cuts")
+	)
 	(gr_arc
 		(start 246.5875 103.125)
@@
 	)
 	(gr_line
+		(start 441.075 164.140984)
+		(end 16.9 164.140984)
+		(stroke
+			(width 0.05)
+			(type default)
+		)
+		(layer "Edge.Cuts")
+	)
+	(gr_line
 		(start 218.8 65.525)
 		(end 231.8 65.525)
@@
 	)
 	(gr_line
-		(start 448.067695 164.140984)
-		(end 9.91 164.140984)
-		(stroke
-			(width 0.05)
-			(type default)
-		)
-		(layer "Edge.Cuts")
-	)
-	(gr_line
 		(start 337.8625 127.725)
 		(end 350.8625 127.725)
@@
 		(layer "Edge.Cuts")
 	)
+	(gr_arc
+		(start 446.075 159.140984)
+		(mid 444.610534 162.676518)
+		(end 441.075 164.140984)
+		(stroke
+			(width 0.05)
+			(type default)
+		)
+		(layer "Edge.Cuts")
+	)
 	(gr_line
 		(start 156.1 52.025)
@@
 	(gr_rect
 		(start 407.42 11.94)
-		(end 429.92 30.76)
+		(end 429.92 33.3)
 		(stroke
 			(width 0.05)
@@
 	)
 	(gr_line
-		(start 453.067695 9.88)
-		(end 453.067695 159.140984)
-		(stroke
-			(width 0.05)
-			(type default)
-		)
-		(layer "Edge.Cuts")
-	)
-	(gr_line
 		(start 79.9 28.2125)
 		(end 79.9 41.2125)
@@
 		(layer "Edge.Cuts")
 	)
-	(gr_arc
-		(start 448.067695 4.88)
-		(mid 451.603229 6.344466)
-		(end 453.067695 9.88)
-		(stroke
-			(width 0.05)
-			(type default)
-		)
-		(layer "Edge.Cuts")
-	)
 	(gr_line
 		(start 199.25 52.025)
@@
 		(layer "Edge.Cuts")
 	)
+	(gr_line
+		(start 446.075 9.88)
+		(end 446.075 159.140984)
+		(stroke
+			(width 0.05)
+			(type default)
+		)
+		(layer "Edge.Cuts")
+	)
 	(gr_arc
 		(start 43.6812 127.725)
@@
 	)
 	(gr_arc
-		(start 453.067695 159.140984)
-		(mid 451.603234 162.676526)
-		(end 448.067695 164.140984)
-		(stroke
-			(width 0.05)
-			(type default)
-		)
-		(layer "Edge.Cuts")
-	)
-	(gr_arc
 		(start 250.85 27.7125)
 		(mid 251.203553 27.858947)
@@
 	)
 	(gr_line
-		(start 4.91 159.140984)
-		(end 4.91 9.88)
+		(start 11.9 159.140984)
+		(end 11.9 9.88)
 		(stroke
 			(width 0.05)
@@
 		(filled_areas_thickness no)
 		(fill yes
-			(mode hatch)
 			(thermal_gap 0.5)
 			(thermal_bridge_width 0.5)
 			(island_removal_mode 1)
 			(island_area_min 10)
-			(hatch_thickness 1)
-			(hatch_gap 1.5)
-			(hatch_orientation 45)
-			(hatch_border_algorithm hatch_thickness)
-			(hatch_min_hole_area 0.3)
 		)
 		(polygon
 			(pts
-				(xy 619.88 -15.75) (xy 610.57 431.29) (xy -14.46 436.46) (xy -11.35 -12.64)
+				(xy 462.2546 -12.2174) (xy 459.8416 180.086) (xy 0.9144 179.5272) (xy 1.4478 -10.1346)
 			)
 		)
